Commit message: made changes in  moveit config files

File: mobile_manipulator_description/urdf/mobile_manipulator.xacro (robot description, xacro)
@@ -625,5 +625,5 @@
   <parent link="knuckle_left_1"/>
   <child link="finger_left_2_1"/>
-  <axis xyz="0.0 0.0 -1.0"/>
+  <axis xyz="0.0 0.0 1.0"/>
 </joint>
 </robot>
