Commit message: publishing to /cmd_vel, robot too heavy previously

File: mobile_robot_description/urdf/mobile_robot.xacro (robot description, xacro)
@@ -11,6 +11,6 @@
   <inertial>
     <origin rpy="0 0 0" xyz="1.1880172534914988e-15 1.8117263115745358e-14 0.3472850110892992"/>
-    <mass value="2953.848903151669"/>
-    <inertia ixx="202.347752" ixy="0.0" ixz="0.0" iyy="313.193688" iyz="0.0" izz="348.342085"/>
+    <mass value="295.3848903151669"/>
+    <inertia ixx="20.2347752" ixy="0.0" ixz="0.0" iyy="31.3193688" iyz="0.0" izz="34.8342085"/>
   </inertial>
   <visual>
@@ -136,5 +136,5 @@
   <parent link="base_link"/>
   <child link="wheel_fl_1"/>
-  <axis xyz="0.0 1.0 -0.0"/>
+  <axis xyz="0.0 1.0 0.0"/>
 </joint>
 <joint name="motor_fr" type="continuous">
@@ -142,5 +142,5 @@
   <parent link="base_link"/>
   <child link="wheel_fr_1"/>
-  <axis xyz="0.0 1.0 -0.0"/>
+  <axis xyz="0.0 1.0 0.0"/>
 </joint>
 <joint name="motor_br" type="continuous">
@@ -148,5 +148,5 @@
   <parent link="base_link"/>
   <child link="wheel_br_1"/>
-  <axis xyz="0.0 1.0 -0.0"/>
+  <axis xyz="0.0 1.0 0.0"/>
 </joint>
 <joint name="lidar_joint" type="fixed">
@@ -159,5 +159,5 @@
   <parent link="base_link"/>
   <child link="wheel_bl_1"/>
-  <axis xyz="0.0 1.0 -0.0"/>
+  <axis xyz="0.0 1.0 0.0"/>
 </joint>
 </robot>
